File: haradware/tachometer/tachometer.kicad_sch (KiCad schematic)
At the start: 5 parts, among them U1 RP2040, U2 LM393

Commit message: KiCad編集
Parts:
- removed D1: LED, symbol Device:LED
- removed D2: D_Photo, symbol Device:D_Photo
- removed U1: RP2040, Package_DFN_QFN:QFN-56-1EP_7x7mm_P0.4mm_EP3.2x3.2mm, symbol MCU_RaspberryPi:RP2040
- removed U2: LM393, symbol Comparator:LM393
- added A1: RaspberryPi_Pico, Module:RaspberryPi_Pico_Common_Unspecified, symbol MCU_Module:RaspberryPi_Pico
- added C1: 0.1u, Capacitor_THT:C_Axial_L5.1mm_D3.1mm_P10.00mm_Horizontal, symbol Device:C
- added J1, J2: Conn_01x03_Pin, Connector_JST:JST_PH_B3B-PH-K_1x03_P2.00mm_Vertical, symbol Connector:Conn_01x03_Pin
- added J3: Battery, Connector_JST:JST_PH_B2B-PH-K_1x02_P2.00mm_Vertical, symbol Connector:Conn_01x02_Pin
- added R2, R3: 10k, Resistor_THT:R_Axial_DIN0207_L6.3mm_D2.5mm_P7.62mm_Horizontal, symbol Device:R
- added RV1, RV2: R_Potentiometer, Potentiometer_THT:Potentiometer_Bourns_3296P_Horizontal, symbol Device:R_Potentiometer
- added SW1: SW_SPST, Button_Switch_THT:SW_Slide-03_Wuerth-WS-SLTV_10x2.5x6.4_P2.54mm, symbol Switch:SW_SPST
- added U2: LN393N, Package_DIP:CERDIP-8_W7.62mm_SideBrazed, symbol New_Library:LN393
- R1: value R100 -> 10k; footprint (none) -> Resistor_THT:R_Axial_DIN0207_L6.3mm_D2.5mm_P7.62mm_Horizontal
Connections:
- net at R1.2: now also A1.26 (GPIO20), U2.1 (OUT1)
- net +3V3: now reaches R1.1
- net +3V3: now also A1.36 (3V3), C1.1, J1.3 (Pin_3), J2.3 (Pin_3), RV1.3, RV2.1, U2.8 (VCC)
- new net: RV2.2, U2.6 (IN2(-))
- new net: J3.1 (Pin_1), SW1.2 (B)
- new net: A1.25 (GPIO19), U2.7 (OUT2)
- new net: RV1.2, U2.2 (IN1(-))
- new net: J1.1 (Pin_1), R2.1, U2.3 (IN1(+))
- new net: J2.1 (Pin_1), R3.1, U2.5 (IN2(+))
- new net GND: A1.13 (GND), A1.18 (GND), A1.23 (GND), A1.28 (GND), A1.3 (GND), A1.38 (GND), A1.8 (GND), C1.2, J1.2 (Pin_2), J2.2 (Pin_2), J3.2 (Pin_2), R2.2, R3.2, RV1.1, RV2.3, U2.4 (GND)
- new net VPP: A1.39 (VSYS), SW1.1 (A)
- no-connect marks 48 -> 29

Commit message: kicad編集
Parts:
- U2: value LN393N -> LM393N
Changed lines of the file:
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@@
 		(color 0 0 0 0)
 	)
+	(junction
+		(at 95.25 30.48)
+		(diameter 0)
+		(color 0 0 0 0)
+	)
 	(no_connect
 		(at 39.37 69.85)
@@
 	(wire
 		(pts
+			(xy 57.15 39.37) (xy 57.15 46.99)
+		)
+		(stroke
+			(width 0)
+			(type default)
+		)
+	)
+	(wire
+		(pts
 			(xy 97.79 111.76) (xy 137.16 111.76)
 		)
@@
 	(wire
 		(pts
+			(xy 95.25 30.48) (xy 99.06 30.48)
+		)
+		(stroke
+			(width 0)
+			(type default)
+		)
+	)
+	(wire
+		(pts
 			(xy 102.87 66.04) (xy 102.87 68.58)
 		)
@@
 	(wire
 		(pts
-			(xy 57.15 39.37) (xy 57.15 46.99)
-		)
-		(stroke
-			(width 0)
-			(type default)
-		)
-	)
-	(wire
-		(pts
 			(xy 143.51 105.41) (xy 143.51 106.68)
 		)
@@
 	(wire
 		(pts
+			(xy 95.25 30.48) (xy 95.25 33.02)
+		)
+		(stroke
+			(width 0)
+			(type default)
+		)
+	)
+	(wire
+		(pts
 			(xy 133.35 91.44) (xy 139.7 91.44)
 		)
@@
 	(wire
 		(pts
-			(xy 93.98 30.48) (xy 99.06 30.48)
+			(xy 93.98 30.48) (xy 95.25 30.48)
 		)
 		(stroke
@@
 	)
 	(symbol
+		(lib_id "power:PWR_FLAG")
+		(at 95.25 33.02 180)
+		(unit 1)
+		(exclude_from_sim no)
+		(in_bom yes)
+		(on_board yes)
+		(dnp no)
+		(fields_autoplaced yes)
+		(property "Reference" "#FLG02"
+			(at 95.25 34.925 0)
+			(effects
+				(font
+					(size 1.27 1.27)
+				)
+				(hide yes)
+			)
+		)
+		(property "Value" "PWR_FLAG"
+			(at 95.25 38.1 0)
+			(effects
+				(font
+					(size 1.27 1.27)
+				)
+			)
+		)
+		(property "Footprint" ""
+			(at 95.25 33.02 0)
+			(effects
+				(font
+					(size 1.27 1.27)
+				)
+				(hide yes)
+			)
+		)
+		(property "Datasheet" "~"
+			(at 95.25 33.02 0)
+			(effects
+				(font
+					(size 1.27 1.27)
+				)
+				(hide yes)
+			)
+		)
+		(property "Description" "Special symbol for telling ERC where power comes from"
+			(at 95.25 33.02 0)
+			(effects
+				(font
+					(size 1.27 1.27)
+				)
+				(hide yes)
+			)
+		)
+		(pin "1"
+		)
+		(instances
+			(project ""
+				(path "/7b2aac6b-0f94-41ef-b71d-7717d821d57e"
+					(reference "#FLG02")
+					(unit 1)
+				)
+			)
+		)
+	)
+	(symbol
 		(lib_id "power:VPP")
 		(at 57.15 39.37 0)
@@
 			)
 		)
-		(property "Value" "LN393N"
+		(property "Value" "LM393N"
 			(at 122.555 78.74 0)
 			(effects

Commit message: 修正して再発注
Parts:
- added D101: Power, LED_THT:LED_D5.0mm, symbol Device:LED
- added J101: OUT_EX, Connector_PinHeader_2.54mm:PinHeader_1x02_P2.54mm_Vertical, symbol Connector_Generic:Conn_01x02
- added J105: Power_EX, Connector_PinHeader_2.54mm:PinHeader_1x02_P2.54mm_Vertical, symbol Connector_Generic:Conn_01x02
- added R101: 10k, Resistor_THT:R_Axial_DIN0207_L6.3mm_D2.5mm_P7.62mm_Horizontal, symbol Device:R
- added R105: 4.7k, Resistor_THT:R_Axial_DIN0207_L6.3mm_D2.5mm_P7.62mm_Horizontal, symbol Device:R
- J103: renamed from J2; value Conn_01x03_Pin -> ch2
- J104: renamed from J1; value Conn_01x03_Pin -> ch1
- renumbered A1 to A101, C1 to C101, J3 to J102, R1 to R102, R2 to R103, R3 to R104, RV2 to RV101, RV1 to RV102, SW1 to SW101, U2 to U101
Connections:
- net +3V3: now also D101.2 (A), J105.1 (Pin_1), R101.1
- net GND: now also J105.2 (Pin_2), R105.2
- net at A101.25 (GPIO19), U101.7 (OUT2): now also J101.2 (Pin_2), R101.2
- net at A101.26 (GPIO20), R102.2, U101.1 (OUT1): now also J101.1 (Pin_1)
- new net: D101.1 (K), R105.1
Other:
- moved on the sheet: C101
