File: haradware/Tachometer_SMD/untitled.kicad_sch (KiCad schematic)
At the start: 9 parts, among them U101 LM393N

Commit message: フットプリント割り当て
Parts:
- C102: footprint (none) -> Capacitor_SMD:C_0402_1005Metric
- C103: footprint (none) -> Capacitor_SMD:C_0201_0603Metric
- D102: footprint (none) -> LED_SMD:LED_0805_2012Metric
- R106, R107, R108: footprint (none) -> Resistor_SMD:R_0402_1005Metric
- RV103, RV104: footprint (none) -> Potentiometer_THT:Potentiometer_Bourns_3296P_Horizontal
- U101: footprint Package_DIP:CERDIP-8_W7.62mm_SideBrazed -> Package_SO:JEITA_SOIC-8_3.9x4.9mm_P1.27mm
Changed lines of the file:
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@@
 			)
 		)
-		(property "Footprint" ""
+		(property "Footprint" "Resistor_SMD:R_0402_1005Metric"
 			(at 88.392 82.55 90)
 			(effects
@@
 			)
 		)
-		(property "Footprint" ""
+		(property "Footprint" "Resistor_SMD:R_0402_1005Metric"
 			(at 76.962 114.3 90)
 			(effects
@@
 			)
 		)
-		(property "Footprint" ""
+		(property "Footprint" "LED_SMD:LED_0805_2012Metric"
 			(at 78.74 104.14 0)
 			(effects
@@
 			)
 		)
-		(property "Footprint" ""
+		(property "Footprint" "Potentiometer_THT:Potentiometer_Bourns_3296P_Horizontal"
 			(at 163.83 100.33 0)
 			(effects
@@
 			)
 		)
-		(property "Footprint" ""
+		(property "Footprint" "Capacitor_SMD:C_0402_1005Metric"
 			(at 106.3752 111.76 0)
 			(effects
@@
 			)
 		)
-		(property "Footprint" ""
+		(property "Footprint" "Potentiometer_THT:Potentiometer_Bourns_3296P_Horizontal"
 			(at 57.15 64.77 0)
 			(effects
@@
 			)
 		)
-		(property "Footprint" ""
+		(property "Footprint" "Resistor_SMD:R_0402_1005Metric"
 			(at 141.478 115.57 90)
 			(effects
@@
 			)
 		)
-		(property "Footprint" "Package_DIP:CERDIP-8_W7.62mm_SideBrazed"
+		(property "Footprint" "Package_SO:JEITA_SOIC-8_3.9x4.9mm_P1.27mm"
 			(at 129.54 93.98 0)
 			(effects
@@
 			)
 		)
-		(property "Footprint" ""
+		(property "Footprint" "Capacitor_SMD:C_0201_0603Metric"
 			(at 91.1352 110.49 0)
 			(effects
